File: STM32_SMD_Quadcopter/_saved_STM32_SMD_Quadcopter.sch (KiCad schematic (older format))
At the start: 66 parts, among them J1 PWR, J2 USB_B_Micro, J3 Micro_SD_Card, J4 DEBUG, M1 Brushed_DC, M2 Brushed_DC, M3 Brushed_DC, M4 Brushed_DC, Q1 IRLML6244TR, Q2 IRLML6244TR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

Commit message: regulator, power over USB, compact SMD, 0603 min cap size
Parts:
- removed C10, C12: 100nF, Capacitor_SMD:C_0402_1005Metric, symbol Device:C_Small
- removed J?: Conn_01x04, symbol Connector_Generic:Conn_01x04
- removed J? (x2): Conn_01x05, symbol Connector_Generic:Conn_01x05
- removed J?: Conn_01x03, symbol Connector_Generic:Conn_01x03
- removed J?: Conn_01x06, symbol Connector_Generic:Conn_01x06
- removed L2: 0.1uH, Inductor_SMD:L_0603_1608Metric, symbol Device:L_Small
- removed R2, R4: 10K, Resistor_SMD:R_0603_1608Metric, symbol Device:R_Small
- removed U1: LM1085-3.3, Connector_PinHeader_2.54mm:PinHeader_1x03_P2.54mm_Vertical, symbol Regulator_Linear:LF33_TO220
- added C10: 100nF, Capacitor_SMD:C_0603_1608Metric, symbol Device:C
- added U1: LT1129-3.3_SOT223, Package_TO_SOT_SMD:SOT-223-3_TabPin2, symbol Regulator_Linear:LT1129-3.3_SOT223
- C1, C11, C17, C18, C19, C2, C20, C21, C22, C7, C8, C9: footprint Capacitor_SMD:C_0402_1005Metric -> Capacitor_SMD:C_0603_1608Metric
- C3, C4: footprint Capacitor_SMD:C_1210_3225Metric -> Capacitor_SMD:C_Elec_3x5.4
- C5: footprint Capacitor_SMD:C_0805_2012Metric -> Capacitor_SMD:C_1210_3225Metric
- J1: footprint Connector_PinHeader_2.54mm:PinHeader_1x02_P2.54mm_Horizontal -> Connector_PinHeader_2.54mm:PinHeader_1x02_P2.54mm_Vertical
Connections:
- net labels added: VUSB
- net labels removed: USB_VBUS
- wire segments 250 -> 242
- no-connect marks 12 -> 42
Other:
- moved on the sheet: C13, C22, C5, D7, D8, J2, J4, R15, R16, U3
