File: STM32_SMD_Quadcopter/STM32_SMD_Quadcopter.sch (KiCad schematic (older format))
At the start: 61 parts, among them J1 PWR, J2 USB_B_Micro, J3 Micro_SD_Card, J4 DEBUG, M1 Brushed_DC, M2 Brushed_DC, M3 Brushed_DC, M4 Brushed_DC, Q1 IRLML6244TR, Q2 IRLML6244TR, Q3 IRLML6244TR, Q4 IRLML6244TR, SW1 SW_Push, U1 LM1085-3.3, U2 MPU-9250, U3 FT230XQ, U4 STM32F446RETx, Y1 8MHz

Commit message: regulator, power over USB, compact SMD, 0603 min cap size
Parts:
- removed C10, C12: 100nF, Capacitor_SMD:C_0402_1005Metric, symbol Device:C_Small
- removed L2: 0.1uH, Inductor_SMD:L_0603_1608Metric, symbol Device:L_Small
- removed R2, R4: 10K, Resistor_SMD:R_0603_1608Metric, symbol Device:R_Small
- removed U1: LM1085-3.3, Connector_PinHeader_2.54mm:PinHeader_1x03_P2.54mm_Vertical, symbol Regulator_Linear:LF33_TO220
- added C10: 100nF, Capacitor_SMD:C_0603_1608Metric, symbol Device:C
- added U1: LT1129-3.3_SOT223, Package_TO_SOT_SMD:SOT-223-3_TabPin2, symbol Regulator_Linear:LT1129-3.3_SOT223
- C1, C11, C17, C18, C19, C2, C20, C21, C22, C7, C8, C9: footprint Capacitor_SMD:C_0402_1005Metric -> Capacitor_SMD:C_0603_1608Metric
- C3, C4: footprint Capacitor_SMD:C_1210_3225Metric -> Capacitor_SMD:C_Elec_3x5.4
- C5: footprint Capacitor_SMD:C_0805_2012Metric -> Capacitor_SMD:C_1210_3225Metric
- J1: footprint Connector_PinHeader_2.54mm:PinHeader_1x02_P2.54mm_Horizontal -> Connector_PinHeader_2.54mm:PinHeader_1x02_P2.54mm_Vertical
Connections:
- net labels added: VUSB
- net labels removed: USB_VBUS
- wire segments 250 -> 242
- no-connect marks 12 -> 42
Other:
- moved on the sheet: C13, C22, C5, D7, D8, J2, J4, R15, R16

Commit message: Latest model, no traces, old crystal
Parts:
- added J5: DSMX, Connector_PinHeader_2.54mm:PinHeader_1x03_P2.54mm_Vertical, symbol Connector_Generic:Conn_01x03
- added R2: 220, Resistor_SMD:R_0603_1608Metric, symbol Device:R
- added R4: 3K, Resistor_SMD:R_0603_1608Metric, symbol Device:R
- added R5: 10K, Resistor_SMD:R_0603_1608Metric, symbol Device:R
- J4: footprint Connector_PinSocket_2.54mm:PinSocket_1x04_P2.54mm_Vertical -> Connector_PinHeader_2.54mm:PinHeader_1x04_P2.54mm_Vertical
- R7, R8: value R -> 470
- Y1: value 8MHz -> 8MHz ECS801830JGNTR; footprint Crystal:Crystal_HC52-U_Vertical -> Crystal:Crystal_SMD_Abracon_ABM3-2Pin_5.0x3.2mm_HandSoldering
Connections:
- net labels added: DSMX, VSENSE
- wire segments 242 -> 255
- no-connect marks 42 -> 40
Other:
- note added: "Other possible FETS:\n\nDMN2041L"
- note added: "Possible alternate: NCP161\n"
Changed lines of the file:
@@
 P 1550 2500
 F 0 "R7" V 1343 2500 50  0000 C CNN
-F 1 "R" V 1434 2500 50  0000 C CNN
+F 1 "470" V 1434 2500 50  0000 C CNN
 F 2 "Resistor_SMD:R_0603_1608Metric" V 1480 2500 50  0001 C CNN
 F 3 "~" H 1550 2500 50  0001 C CNN
@@
 P 1550 3000
 F 0 "R8" V 1343 3000 50  0000 C CNN
-F 1 "R" V 1434 3000 50  0000 C CNN
+F 1 "470" V 1434 3000 50  0000 C CNN
 F 2 "Resistor_SMD:R_0603_1608Metric" V 1480 3000 50  0001 C CNN
 F 3 "~" H 1550 3000 50  0001 C CNN
@@
 P 7750 4400
 F 0 "Y1" V 7704 4531 50  0000 L CNN
-F 1 "8MHz" V 7795 4531 50  0000 L CNN
-F 2 "Crystal:Crystal_HC52-U_Vertical" H 7750 4400 50  0001 C CNN
+F 1 "8MHz ECS801830JGNTR" V 7600 4200 50  0000 L CNN
+F 2 "Crystal:Crystal_SMD_Abracon_ABM3-2Pin_5.0x3.2mm_HandSoldering" H 7750 4400 50  0001 C CNN
 F 3 "~" H 7750 4400 50  0001 C CNN
 	1    7750 4400
@@
 F 0 "J4" H 6472 5380 50  0000 R CNN
 F 1 "DEBUG" H 6472 5471 50  0000 R CNN
-F 2 "Connector_PinSocket_2.54mm:PinSocket_1x04_P2.54mm_Vertical" H 6500 5500 50  0001 C CNN
+F 2 "Connector_PinHeader_2.54mm:PinHeader_1x04_P2.54mm_Vertical" H 6500 5500 50  0001 C CNN
 F 3 "~" H 6500 5500 50  0001 C CNN
 	1    6500 5500
@@
 NoConn ~ 9700 3450
 NoConn ~ 9700 3550
-NoConn ~ 9700 4450
 NoConn ~ 9700 4750
 NoConn ~ 9700 5050
@@
 NoConn ~ 8300 5350
 NoConn ~ 8300 5250
-NoConn ~ 8300 5150
 NoConn ~ 8300 4650
 Wire Wire Line
@@
 	1    0    0    -1
 $EndComp
+$Comp
+L Connector_Generic:Conn_01x03 J5
+U 1 1 5E9FBB50
+P 5100 3200
+F 0 "J5" H 5179 3242 50  0000 L CNN
+F 1 "DSMX" H 5179 3151 50  0000 L CNN
+F 2 "Connector_PinHeader_2.54mm:PinHeader_1x03_P2.54mm_Vertical" H 5100 3200 50  0001 C CNN
+F 3 "~" H 5100 3200 50  0001 C CNN
+	1    5100 3200
+	1    0    0    -1
+$EndComp
+$Comp
+L power:GND #PWR047
+U 1 1 5E9FCBCD
+P 4800 3350
+F 0 "#PWR047" H 4800 3100 50  0001 C CNN
+F 1 "GND" H 4805 3177 50  0000 C CNN
+F 2 "" H 4800 3350 50  0001 C CNN
+F 3 "" H 4800 3350 50  0001 C CNN
+	1    4800 3350
+	1    0    0    -1
+$EndComp
+$Comp
+L power:+3.3V #PWR031
+U 1 1 5E9FCCA2
+P 4800 3050
+F 0 "#PWR031" H 4800 2900 50  0001 C CNN
+F 1 "+3.3V" H 4815 3223 50  0000 C CNN
+F 2 "" H 4800 3050 50  0001 C CNN
+F 3 "" H 4800 3050 50  0001 C CNN
+	1    4800 3050
+	1    0    0    -1
+$EndComp
+Wire Wire Line
+	4800 3050 4800 3200
+Wire Wire Line
+	4800 3200 4900 3200
+Wire Wire Line
+	4800 3350 4800 3300
+Wire Wire Line
+	4800 3300 4900 3300
+Wire Wire Line
+	4900 3100 4750 3100
+$Comp
+L Device:R R2
+U 1 1 5EA2C14D
+P 4600 3100
+F 0 "R2" V 4393 3100 50  0000 C CNN
+F 1 "220" V 4484 3100 50  0000 C CNN
+F 2 "Resistor_SMD:R_0603_1608Metric" V 4530 3100 50  0001 C CNN
+F 3 "~" H 4600 3100 50  0001 C CNN
+	1    4600 3100
+	0    1    1    0
+$EndComp
+Wire Wire Line
+	4450 3100 4350 3100
+Text GLabel 8250 5150 0    50   Input ~ 0
+DSMX
+Wire Wire Line
+	8250 5150 8300 5150
+Text GLabel 4350 3100 0    50   Input ~ 0
+DSMX
+Text GLabel 9750 4450 2    50   Input ~ 0
+VSENSE
+Wire Wire Line
+	9750 4450 9700 4450
+Text GLabel 6000 3250 2    50   Input ~ 0
+VSENSE
+$Comp
+L Device:R R4
+U 1 1 5EA7F42D
+P 5900 3050
+F 0 "R4" H 5970 3096 50  0000 L CNN
+F 1 "3K" H 5970 3005 50  0000 L CNN
+F 2 "Resistor_SMD:R_0603_1608Metric" V 5830 3050 50  0001 C CNN
+F 3 "~" H 5900 3050 50  0001 C CNN
+	1    5900 3050
+	1    0    0    -1
+$EndComp
+$Comp
+L Device:R R5
+U 1 1 5EA7F4C7
+P 5900 3450
+F 0 "R5" H 5970 3496 50  0000 L CNN
+F 1 "10K" H 5970 3405 50  0000 L CNN
+F 2 "Resistor_SMD:R_0603_1608Metric" V 5830 3450 50  0001 C CNN
+F 3 "~" H 5900 3450 50  0001 C CNN
+	1    5900 3450
+	1    0    0    -1
+$EndComp
+Wire Wire Line
+	5900 3200 5900 3250
+Wire Wire Line
+	6000 3250 5900 3250
+Connection ~ 5900 3250
+Wire Wire Line
+	5900 3250 5900 3300
+$Comp
+L power:GND #PWR049
+U 1 1 5EAA08C9
+P 5900 3650
+F 0 "#PWR049" H 5900 3400 50  0001 C CNN
+F 1 "GND" H 5905 3477 50  0000 C CNN
+F 2 "" H 5900 3650 50  0001 C CNN
+F 3 "" H 5900 3650 50  0001 C CNN
+	1    5900 3650
+	1    0    0    -1
+$EndComp
+Wire Wire Line
+	5900 3600 5900 3650
+Wire Wire Line
+	5900 2900 5900 2850
+$Comp
+L power:+BATT #PWR048
+U 1 1 5EAC295D
+P 5900 2850
+F 0 "#PWR048" H 5900 2700 50  0001 C CNN
+F 1 "+BATT" H 5915 3023 50  0000 C CNN
+F 2 "" H 5900 2850 50  0001 C CNN
+F 3 "" H 5900 2850 50  0001 C CNN
+	1    5900 2850
+	1    0    0    -1
+$EndComp
+Text Notes 1700 6350 0    50   ~ 0
+Other possible FETS:\n\nDMN2041L
+Text Notes 1650 2150 0    50   ~ 0
+Possible alternate: NCP161\n
 $EndSCHEMATC

Commit message: Made much denser, added traces
Parts:
- J2: footprint Connector_USB:USB_Micro-B_Amphenol_10103594-0001LF_Horizontal -> Connector_USB:USB_Micro-B_Molex_47346-0001
- J3: footprint Connector_Card:microSD_HC_Wuerth_693072010801 -> Connector_Card:microSD_HC_Hirose_DM3D-SF; symbol Connector:Micro_SD_Card -> STM32_SMD_Quadcopter-rescue:Micro_SD_Card-Connector
- U3: symbol Interface_USB:FT230XQ -> STM32_SMD_Quadcopter-rescue:FT230XQ-Interface_USB
Changed lines of the file:
@@
 EESchema Schematic File Version 4
-LIBS:STM32_SMD_Quadcopter-cache
-EELAYER 26 0
+EELAYER 30 0
 EELAYER END
 $Descr A 11000 8500
@@
 	900  3000 950  3000
 $Comp
-L Connector:Micro_SD_Card J3
+L STM32_SMD_Quadcopter-rescue:Micro_SD_Card-Connector J3
 U 1 1 5D1D8D5D
 P 5200 5000
 F 0 "J3" H 5150 5717 50  0000 C CNN
 F 1 "Micro_SD_Card" H 5150 5626 50  0000 C CNN
-F 2 "Connector_Card:microSD_HC_Wuerth_693072010801" H 6350 5300 50  0001 C CNN
+F 2 "Connector_Card:microSD_HC_Hirose_DM3D-SF" H 6350 5300 50  0001 C CNN
 F 3 "http://katalog.we-online.de/em/datasheet/693072010801.pdf" H 5200 5000 50  0001 C CNN
 	1    5200 5000
@@
 F 0 "J2" H 5570 1598 50  0000 R CNN
 F 1 "USB_B_Micro" H 5570 1689 50  0000 R CNN
-F 2 "Connector_USB:USB_Micro-B_Amphenol_10103594-0001LF_Horizontal" H 5950 1650 50  0001 C CNN
+F 2 "Connector_USB:USB_Micro-B_Molex_47346-0001" H 5950 1650 50  0001 C CNN
 F 3 "~" H 5950 1650 50  0001 C CNN
 	1    5800 1700
@@
 	9700 4350 9750 4350
 Text GLabel 1050 4300 0    50   Input ~ 0
-SPI1_SCK
+SPI2_SCK
 Text GLabel 1050 4200 0    50   Input ~ 0
-SPI1_MISO
+SPI2_MISO
 Text GLabel 1050 4100 0    50   Input ~ 0
-SPI1_MOSI
+SPI2_MOSI
 Wire Wire Line
 	2150 3500 2350 3500
@@
 	3100 4500 3100 4700
 Text GLabel 4250 4900 0    50   Input ~ 0
-SPI2_MOSI
+SPI1_MOSI
 Text GLabel 4250 5300 0    50   Input ~ 0
-SPI2_MISO
+SPI1_MISO
 Text GLabel 4250 5100 0    50   Input ~ 0
-SPI2_SCK
+SPI1_SCK
 NoConn ~ 4300 4700
 Text GLabel 4250 4800 0    50   Input ~ 0
@@
 Wire Wire Line
 	4250 5300 4300 5300
+Text GLabel 9750 3650 2    50   Input ~ 0
+SD_CARD_CS
+Wire Wire Line
+	8250 4850 8300 4850
 Text GLabel 8250 4850 0    50   Input ~ 0
-SD_CARD_CS
-Wire Wire Line
-	8250 4850 8300 4850
-Text GLabel 9750 3650 2    50   Input ~ 0
 MPU9250_CS
 Wire Wire Line
@@
 USART1_RX
 $Comp
-L Interface_USB:FT230XQ U3
+L STM32_SMD_Quadcopter-rescue:FT230XQ-Interface_USB U3
 U 1 1 5D7FF237
 P 7350 1700
@@
 NoConn ~ 9700 5150
 NoConn ~ 9700 5350
-NoConn ~ 9700 5450
 NoConn ~ 9700 6050
 NoConn ~ 9700 6150
@@
 Wire Wire Line
 	4450 3100 4350 3100
-Text GLabel 8250 5150 0    50   Input ~ 0
+Text GLabel 9750 5450 2    50   Input ~ 0
 DSMX
-Wire Wire Line
-	8250 5150 8300 5150
 Text GLabel 4350 3100 0    50   Input ~ 0
 DSMX
@@
 Text Notes 1650 2150 0    50   ~ 0
 Possible alternate: NCP161\n
+Wire Wire Line
+	9750 5450 9700 5450
+NoConn ~ 8300 5150
 $EndSCHEMATC

Commit message: Completed board v1
Parts:
- removed J3: Micro_SD_Card, Connector_Card:microSD_HC_Hirose_DM3D-SF, symbol STM32_SMD_Quadcopter-rescue:Micro_SD_Card-Connector
- added J3: Micro_SD_Card_Det, Connector_Card:microSD_HC_Hirose_DM3D-SF, symbol Connector:Micro_SD_Card_Det
- J4: footprint Connector_PinHeader_2.54mm:PinHeader_1x04_P2.54mm_Vertical -> Connector_Harwin:Harwin_M20-89004xx_1x04_P2.54mm_Horizontal
Connections:
- net +3V3: now also J3.4 (VDD)
- net GND: now also J3.10 (DET_A), J3.11 (SHIELD), J3.6 (VSS), J3.9 (DET_B)
- net SD_CARD_CS: now also J3.2 (DAT3/CD)
- net SPI1_MISO: now also J3.7 (DAT0)
- net SPI1_MOSI: now also J3.3 (CMD)
- net SPI1_SCK: now also J3.5 (CLK)
Changed lines of the file:
@@
 	900  3000 950  3000
-$Comp
-L STM32_SMD_Quadcopter-rescue:Micro_SD_Card-Connector J3
-U 1 1 5D1D8D5D
-P 5200 5000
-F 0 "J3" H 5150 5717 50  0000 C CNN
-F 1 "Micro_SD_Card" H 5150 5626 50  0000 C CNN
-F 2 "Connector_Card:microSD_HC_Hirose_DM3D-SF" H 6350 5300 50  0001 C CNN
-F 3 "http://katalog.we-online.de/em/datasheet/693072010801.pdf" H 5200 5000 50  0001 C CNN
-	1    5200 5000
-	1    0    0    -1
-$EndComp
 $Comp
 L Connector:USB_B_Micro J2
@@
 F 0 "J4" H 6472 5380 50  0000 R CNN
 F 1 "DEBUG" H 6472 5471 50  0000 R CNN
-F 2 "Connector_PinHeader_2.54mm:PinHeader_1x04_P2.54mm_Vertical" H 6500 5500 50  0001 C CNN
+F 2 "Connector_Harwin:Harwin_M20-89004xx_1x04_P2.54mm_Horizontal" H 6500 5500 50  0001 C CNN
 F 3 "~" H 6500 5500 50  0001 C CNN
 	1    6500 5500
@@
 	9750 5450 9700 5450
 NoConn ~ 8300 5150
+$Comp
+L Connector:Micro_SD_Card_Det J3
+U 1 1 5EAFBA60
+P 5200 5100
+F 0 "J3" H 5150 5917 50  0000 C CNN
+F 1 "Micro_SD_Card_Det" H 5150 5826 50  0000 C CNN
+F 2 "Connector_Card:microSD_HC_Hirose_DM3D-SF" H 7250 5800 50  0001 C CNN
+F 3 "https://www.hirose.com/product/en/download_file/key_name/DM3/category/Catalog/doc_file_id/49662/?file_category_id=4&item_id=195&is_series=1" H 5200 5200 50  0001 C CNN
+	1    5200 5100
+	1    0    0    -1
+$EndComp
+$Comp
+L power:GND #PWR?
+U 1 1 5EB10C43
+P 4200 5700
+F 0 "#PWR?" H 4200 5450 50  0001 C CNN
+F 1 "GND" H 4205 5527 50  0000 C CNN
+F 2 "" H 4200 5700 50  0001 C CNN
+F 3 "" H 4200 5700 50  0001 C CNN
+	1    4200 5700
+	1    0    0    -1
+$EndComp
+Wire Wire Line
+	4200 5700 4200 5600
+Wire Wire Line
+	4200 5600 4300 5600
+Wire Wire Line
+	4300 5500 4200 5500
+Wire Wire Line
+	4200 5500 4200 5600
+Connection ~ 4200 5600
 $EndSCHEMATC

Commit message: V2 started, using different crystal, ICM20948, 10 pin SWD header, and multiple component swaps
Parts:
- removed J4: DEBUG, Connector_Harwin:Harwin_M20-89004xx_1x04_P2.54mm_Horizontal, symbol Connector:Conn_01x04_Male
- removed U1: LT1129-3.3_SOT223, Package_TO_SOT_SMD:SOT-223-3_TabPin2, symbol Regulator_Linear:LT1129-3.3_SOT223
- removed U2: MPU-9250, Sensor_Motion:InvenSense_QFN-24_3x3mm_P0.4mm, symbol Sensor_Motion:MPU-9250
- removed Y1: 8MHz ECS801830JGNTR, Crystal:Crystal_SMD_Abracon_ABM3-2Pin_5.0x3.2mm_HandSoldering, symbol Device:Crystal
- added C12, C14, C23: 2.2uF, Capacitor_SMD:C_0603_1608Metric, symbol Device:C_Small
- added C15: 4.7uF, Capacitor_SMD:C_1210_3225Metric, symbol Device:C
- added C16: 100nF, Capacitor_SMD:C_0603_1608Metric, symbol Device:C_Small
- added J4: DEBUG, Connector_PinSocket_1.27mm:PinSocket_2x05_P1.27mm_Vertical_SMD, symbol Connector_Generic:Conn_02x05_Odd_Even
- added Q5, Q6, Q7, Q8: 2N7002, Package_TO_SOT_SMD:SOT-23, symbol Transistor_FET:2N7002
- added R18, R19, R20, R21, R22, R23, R24, R6: 10K, Resistor_SMD:R_0603_1608Metric, symbol Device:R_Small
- added R25: 22, Resistor_SMD:R_0603_1608Metric, symbol Device:R
- added U1: AMS1117-3.3, Package_TO_SOT_SMD:SOT-223-3_TabPin2, symbol Regulator_Linear:AMS1117-3.3
- added U2: AMS1117-1.8, Package_TO_SOT_SMD:SOT-223-3_TabPin2, symbol Regulator_Linear:AMS1117-1.8
- added U5: ICM-20948, Sensor_Motion:InvenSense_QFN-24_3x3mm_P0.4mm, symbol Sensor_Motion:ICM-20948
- added Y1: 16MHz X322516MLB4SI, Crystal:Crystal_SMD_3225-4Pin_3.2x2.5mm, symbol Device:Crystal_GND24_Small
- C20, C21: value 22pF -> 12pF
- J2: symbol Connector:USB_B_Micro -> STM32_SMD_Quadcopter-rescue:USB_B_Micro-Connector
- R15, R16: value 300 -> 2K
- R4: value 3K -> 30K
- R5: value 10K -> 100K
- R7, R8: value 470 -> 4.7k
Connections:
- net +3V3: now also C14.2, J4.1 (Pin_1), R21.1, R22.1, R23.1, R24.1, R25.2, U1.2 (VO), U2.3 (VI), U5.13 (VDD); no longer C10.2, U3.8 (3V3OUT), U3.9 (~RESET)
- net +BATT: now also U1.3 (VI)
- net GND: now also C20.2, C21.2, C12.1, C14.1, C15.2, C16.2, C23.1, J4.3 (Pin_3), J4.5 (Pin_5), J4.9 (Pin_9), U1.1 (GND), U2.1 (GND), U5.18 (GND), U5.20 (GND), Y1.2, Y1.4; no longer C20.1, C21.1
- net MPU9250_CS: now also Q8.3 (D), R24.2
- net SPI2_MISO: now also Q5.3 (D), R21.2
- net SPI2_MOSI: now also Q6.3 (D), R22.2
- net SPI2_SCK: now also Q7.3 (D), R23.2
- net SYS_JTCL-SWCLK: now also J4.4 (Pin_4)
- net SYS_JTMS-SWDIO: now also J4.2 (Pin_2)
- net at C7.1: now also U5.10 (REGOUT)
- net at U4.5 (PH0): now also C20.1, Y1.1; no longer C20.2
- net at U4.6 (PH1): now also C21.1, Y1.3; no longer C21.2
- net NRST: now reaches R17.2, SW1.2, U4.7 (NRST)
- net NRST: now also C23.2, J4.10 (Pin_10)
- new net: C10.2, R25.1, U3.8 (3V3OUT), U3.9 (~RESET)
- new net +1V8: C12.2, C15.1, C16.1, Q5.1 (G), Q6.1 (G), Q7.1 (G), Q8.1 (G), R18.1, R19.1, R20.1, R6.1, U2.2 (VO), U5.8 (VDDIO)
- new net MPU9250_CS_1.8V: Q8.2 (S), R20.2, U5.22 (~CS)
- new net SPI2_MISO_1.8V: Q5.2 (S), R6.2, U5.9 (SDO/AD0)
- new net SPI2_MOSI_1.8V: Q6.2 (S), R18.2, U5.24 (SDA/SDI)
- new net SPI2_SCK_1.8V: Q7.2 (S), R19.2, U5.23 (SCL/SCLK)
- no-connect marks 40 -> 43
Other:
- note added: "Possible alternate: \nNCP161\nLT1129"
- note removed: "Possible alternate: NCP161\n"
- moved on the sheet: C1, C10, C11, C13, C17, C18, C19, C2, C22, C3, C4, C5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

Commit message: All parts set in place
Parts:
- removed C11: 100nF, Capacitor_SMD:C_0603_1608Metric, symbol Device:C_Small
- removed C12, C14, C23: 2.2uF, Capacitor_SMD:C_0603_1608Metric, symbol Device:C_Small
- removed C13: 100uF, Capacitor_SMD:C_1210_3225Metric, symbol Device:C
- removed C15: 4.7uF, Capacitor_SMD:C_1210_3225Metric, symbol Device:C
- removed C4: 100uF, Capacitor_SMD:C_Elec_3x5.4, symbol Device:C
- removed Q6, Q7, Q8: 2N7002, Package_TO_SOT_SMD:SOT-23, symbol Transistor_FET:2N7002
- C1, C10, C16, C17, C2, C7, C8, C9: footprint Capacitor_SMD:C_0603_1608Metric -> Capacitor_SMD:C_0402_1005Metric
- R18, R20, R22: value 10K -> 1K; footprint Resistor_SMD:R_0603_1608Metric -> Resistor_SMD:R_0402_1005Metric
- R19, R23, R24: value 10K -> 1.2K; footprint Resistor_SMD:R_0603_1608Metric -> Resistor_SMD:R_0402_1005Metric
- R21, R25, R6: footprint Resistor_SMD:R_0603_1608Metric -> Resistor_SMD:R_0402_1005Metric
Connections:
- net +1V8: no longer R18.1, R19.1, R20.1
- net +3V3: no longer R22.1, R23.1, R24.1
- net GND: now also R19.2, R23.2, R24.2
- net MPU9250_CS: now also R20.1; no longer R24.2
- net MPU9250_CS_1.8V: now also R24.1
- net SPI2_MOSI: now also R18.1; no longer R22.2
- net SPI2_MOSI_1.8V: now also R19.1
- net SPI2_SCK: now also R22.1; no longer R23.2
- net SPI2_SCK_1.8V: now also R22.2, R23.1; no longer R19.2
Other:
- moved on the sheet: C16, C3, C5, C6, C9, R20, R24, U1, U2
